Commit message: Resuelto el problema de las ruedas, ahora hay que agregar una camara al modelo (y quizas un lidar) y configurar los momentos de inercia si pinta.

File: model.xacro (robot description, xacro)
@@ -61,6 +61,8 @@
 	</link>
 	<xacro:macro name="wheel" params="name pos">
+		<xacro:property name="position" value="0.1 ${pos*0.17} -0.037" />
+		<xacro:property name="position2" value="0 0 0" />
+		<xacro:property name="orientation" value="0 1.5707 1.570" />
 		<link name="${name}_wheel">
-			<origin xyz="0.1 ${pos} 0.11" rpy="0 1.5707 1.5707"/>
 			<inertial>
 				<mass value="1.5"/>
@@ -68,4 +70,5 @@
 			</inertial>
 			<collision name="collision">
+				<origin xyz="${position2}" rpy="${orientation}"/>
 				<geometry>
 					<cylinder radius="0.11" length="0.05"/>
@@ -83,4 +86,5 @@
 			</collision>
 			<visual name="${name}_visual">
+				<origin xyz="${position2}" rpy="${orientation}"/>
 				<geometry>
 					<cylinder radius="0.11" length="0.05"/>
@@ -97,21 +101,14 @@
       </visual>
     </link>
-    </xacro:macro>
-    <xacro:wheel name="right" pos="0.17" />
-    <xacro:wheel name="left" pos="-0.17" />
-    <joint type="revolute" name="left_wheel_hinge">
-	    <origin xyz="0 0 -0.03" rpy="0 0 0"/>
-	    <child link="left_wheel"/>
+    <joint type="revolute" name="${name}_wheel_hinge">
+	    <origin xyz="${position}" rpy="0 0 0"/>
+	    <child link="${name}_wheel"/>
 	    <parent link="chassis"/>
 	    <axis xyz="0 1 0"/>
 	    <limit effort="30" velocity="1" lower="-7" upper="7" />
     </joint>
-    <joint type="revolute" name="right_wheel_hinge">
-	    <origin xyz="0 0 0.03" rpy="0 0 0"/>
-	    <child link="right_wheel"/>
-	    <parent link="chassis"/>
-	    <axis xyz="0 1 0"/>
-	    <limit effort="30" velocity="1.0" lower="-7" upper="7"/>
-    </joint>
+    </xacro:macro>
+    <xacro:wheel name="right" pos="1" />
+    <xacro:wheel name="left" pos="-1" />
     <!--
 	    <plugin filename="libDiffDrivePlugin.so" name="diff_drive">

Commit message: camara agregada. Ahora hay que hacer la integración con gazebo y agregarle los pluggins

File: model.xacro (robot description, xacro)
@@ -111,4 +111,20 @@
     <xacro:wheel name="right" pos="1" />
     <xacro:wheel name="left" pos="-1" />
+    <link name="Camera">
+	    <visual name="camera_visual">
+		    <origin xyz="0 0 0" rpy="0 0 0"/>
+		    <geometry>
+			    <box size="0.1 0.1 0.1"/>
+		    </geometry>
+		    <material name="camera_color">
+			    <color rgba="1 1 1 1"/>
+		    </material>
+	    </visual>
+    </link>
+    <joint name="camera_to_chassis" type="fixed">
+	    <parent link="chassis"/>
+	    <child link="Camera"/>
+	    <origin xyz="0.14 0 0.16" rpy="0 0 0" />
+    </joint>
     <!--
 	    <plugin filename="libDiffDrivePlugin.so" name="diff_drive">

Commit message: se agrego el mundo configurado y alguns pluggins. Voy a testear su funcionamiento mediante un nodo de python.

File: model.xacro (robot description, xacro)
@@ -104,10 +104,10 @@
       </visual>
     </link>
-    <joint type="revolute" name="${name}_wheel_hinge">
+    <joint type="continuous" name="${name}_wheel_hinge">
 	    <origin xyz="${position}" rpy="0 0 0"/>
 	    <child link="${name}_wheel"/>
 	    <parent link="chassis"/>
 	    <axis xyz="0 1 0"/>
-	    <limit effort="30" velocity="1" lower="-7" upper="7" />
+	    <!-- <limit effort="30" velocity="1" lower="-7" upper="7" />-->
     </joint>
     </xacro:macro>
@@ -131,44 +131,9 @@
     </joint>
     <!-- Fuente: http://gazebosim.org/tutorials?tut=ros_gzplugins -->
+<!-- Plugins -->
     <!-- camera -->
-  <gazebo reference="Camera">
-    <sensor type="camera" name="camera1">
-      <update_rate>30.0</update_rate>
-      <camera name="head">
-        <horizontal_fov>1.3962634</horizontal_fov>
-        <image>
-          <width>800</width>
-          <height>800</height>
-          <format>R8G8B8</format>
-        </image>
-        <clip>
-          <near>0.02</near>
-          <far>300</far>
-        </clip>
-        <noise>
-          <type>gaussian</type>
-          <!-- Noise is sampled independently per pixel on each frame.
-               That pixel's noise value is added to each of its color
-               channels, which at that point lie in the range [0,1]. -->
-          <mean>0.0</mean>
-          <stddev>0.007</stddev>
-        </noise>
-      </camera>
-      <plugin name="camera_controller" filename="libgazebo_ros_camera.so">
-        <alwaysOn>true</alwaysOn>
-        <updateRate>0.0</updateRate>
-        <cameraName>pioneer2dx/camera1</cameraName>
-        <imageTopicName>image_raw</imageTopicName>
-        <cameraInfoTopicName>camera_info</cameraInfoTopicName>
-        <frameName>camera_link</frameName>
-        <hackBaseline>0.07</hackBaseline>
-        <distortionK1>0.0</distortionK1>
-        <distortionK2>0.0</distortionK2>
-        <distortionK3>0.0</distortionK3>
-        <distortionT1>0.0</distortionT1>
-        <distortionT2>0.0</distortionT2>
-      </plugin>
-    </sensor>
-  </gazebo>
+    <xacro:include filename="camera_plug.xacro"/>
+    <!--<xacro:include filename="differential_plug.xacro"/>
+    <xacro:include filename="transmition.xacro"/>-->
     <!--
 	    <plugin filename="libDiffDrivePlugin.so" name="diff_drive">

Commit message: Se agrego el lidar hokuyo del tutorial de gazebo, se comprobo el funcionamiento en rviz y se agrupo en una carpeta todos los plugins. Hay muchas cosas que corregir y modificar, pero voy por lo significativo por ahora. Tambien se agregó el texto de la licencia

File: model.xacro (robot description, xacro)
@@ -122,10 +122,35 @@
 	    <origin xyz="0.14 0 0.16" rpy="0 0 0" />
     </joint>
+    <link name="Lidar">
+	    <!--<visual name="Lidar_visual">
+		    <origin xyz="0 0 0" rpy="0 0 0"/>
+		    <geometry>
+			    <box size="0.1 0.1 0.1"/>
+		    </geometry>
+		    <material name="Lidar_color">
+			    <color rgba="0 0 1 1"/>
+		    </material>
+	    </visual>-->
+     <visual>
+      <origin xyz="0 0 0" rpy="0 0 0"/>
+      <geometry>
+	      <!-- <mesh filename="package://rrbot_description/meshes/hokuyo.dae"/>-->
+	<mesh filename="file://$(arg meshlocation)/meshes/hokuyo.dae"/>
+      </geometry>
+    </visual>
+    </link>
+    <joint name="lidar_to_chassis" type="fixed">
+	    <parent link="chassis"/>
+	    <child link="Lidar"/>
+	    <axis xyz="0 1 0"/>
+	    <origin xyz="0.14 0 0.4" rpy="0 0 0" />
+    </joint>
     <!-- Fuente: http://gazebosim.org/tutorials?tut=ros_gzplugins -->
 <!-- Plugins -->
     <!-- camera -->
-    <xacro:include filename="camera_plug.xacro"/>
-    <!--<xacro:include filename="differential_plug.xacro"/>
-    <xacro:include filename="transmition.xacro"/>-->
+    <xacro:include filename="./plugins/camera_plug.xacro"/>
+    <xacro:include filename="./plugins/lidar_plug.xacro"/>
+    <!--<xacro:include filename="./plugins/differential_plug.xacro"/>
+    <xacro:include filename="./plugins/transmition.xacro"/>-->
     <!--
 	    <plugin filename="libDiffDrivePlugin.so" name="diff_drive">
