Commit message: Se creo el package para que pueda ser facilmente referenciado

File: models/model.xacro (robot description, xacro)
@@ -42,6 +42,6 @@
 			<origin xyz="0 0 0.04" rpy="0 0 0"/>
 			<geometry>
-				<!--<mesh filename="package://pioneer2dx/meshes/chassis.dae"/>-->
-				<mesh filename="file://$(arg meshlocation)/meshes/chassis.dae"/>
+				<mesh filename="package://pioneer2dx/meshes/chassis.dae"/>
+				<!--<mesh filename="file://$(arg meshlocation)/meshes/chassis.dae"/>-->
 			</geometry>
 		</visual>
@@ -135,6 +135,6 @@
       <origin xyz="0 0 0" rpy="0 0 0"/>
       <geometry>
-	      <!-- <mesh filename="package://rrbot_description/meshes/hokuyo.dae"/>-->
-	<mesh filename="file://$(arg meshlocation)/meshes/hokuyo.dae"/>
+	      <mesh filename="package://pioneer2dx/meshes/hokuyo.dae"/>
+	      <!--<mesh filename="file://$(arg meshlocation)/meshes/hokuyo.dae"/>-->
       </geometry>
     </visual>
@@ -149,6 +149,8 @@
 <!-- Plugins -->
     <!-- camera -->
-    <xacro:include filename="./plugins/camera_plug.xacro"/>
-    <xacro:include filename="./plugins/lidar_plug.xacro"/>
+    <xacro:include filename="$(find pioneer2dx)/plugins/camera_plug.xacro"/>
+    <xacro:include filename="$(find pioneer2dx)/plugins/lidar_plug.xacro"/>
+    <!--<xacro:include filename="./plugins/camera_plug.xacro"/>
+    <xacro:include filename="./plugins/lidar_plug.xacro"/>-->
     <!--<xacro:include filename="./plugins/differential_plug.xacro"/>
     <xacro:include filename="./plugins/transmition.xacro"/>-->
